File: my-template/keyboard_matrix.kicad_sch (KiCad schematic)
At the start: 174 parts, among them SW1 esc, SW10 f9, SW11 f10, SW12 f11, SW13 f12, SW14 prtsc, SW15 scroll lock, SW16 pause break, SW17 ~ `, SW18 ! 1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

Commit message: lipo schematic done
Other:
- title: (none) -> 80% Layout keyboard matrix
Changed lines of the file:
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@@
 	(generator_version "9.0")
 	(paper "User" 431.8 304.8)
+	(title_block
+		(title "80% Layout keyboard matrix")
+	)
 	(junction
 		(at 261.62 194.31)
