File: my-template/my-template.kicad_pcb (KiCad board)
At the start: 2 copper layers, 0 parts

Commit message: component placement done
Parts:
- added C1: C_Small, Capacitor_SMD:C_0603_1608Metric, F.Cu at (176.7, 58.9)
- added C2: C, Capacitor_SMD:C_0603_1608Metric, F.Cu at (173.1, 58.9)
- added C3: C, Capacitor_SMD:C_0603_1608Metric, F.Cu at (169.6, 58.9)
- added C4: C, Capacitor_SMD:C_0603_1608Metric, F.Cu at (183.9, 58.9)
- added C5: C, Capacitor_SMD:C_0603_1608Metric, F.Cu at (180.3, 58.9)
- added CR1: USBLC6-2SC6, myLibrary:USBLC6-2SC6, F.Cu at (74.1, 72.0)
- added D1: D, Diode_SMD:D_SOD-123, B.Cu at (48.7, 96.1)
- added D10: D, Diode_SMD:D_SOD-123, B.Cu at (258.2, 96.1)
- added D11: D, Diode_SMD:D_SOD-123, B.Cu at (277.3, 96.1)
- added D12: D, Diode_SMD:D_SOD-123, B.Cu at (296.3, 96.1)
- added D13: D, Diode_SMD:D_SOD-123, B.Cu at (315.4, 96.1)
- added D14: D, Diode_SMD:D_SOD-123, B.Cu at (339.2, 96.1)
- added D15: D, Diode_SMD:D_SOD-123, B.Cu at (358.2, 96.1)
- added D16: D, Diode_SMD:D_SOD-123, B.Cu at (377.3, 96.1)
- added D17: D, Diode_SMD:D_SOD-123, B.Cu at (48.7, 124.6)
- added D18: D, Diode_SMD:D_SOD-123, B.Cu at (67.7, 124.6)
- added D19: D, Diode_SMD:D_SOD-123, B.Cu at (86.8, 124.6)
- added D2: D, Diode_SMD:D_SOD-123, B.Cu at (86.8, 96.1)
- added D20: D, Diode_SMD:D_SOD-123, B.Cu at (105.8, 124.6)
- added D21: D, Diode_SMD:D_SOD-123, B.Cu at (124.9, 124.6)
- added D22: D, Diode_SMD:D_SOD-123, B.Cu at (143.9, 124.6)
- added D23: D, Diode_SMD:D_SOD-123, B.Cu at (163.0, 124.6)
- added D24: D, Diode_SMD:D_SOD-123, B.Cu at (182.0, 124.6)
- added D25: D, Diode_SMD:D_SOD-123, B.Cu at (201.1, 124.6)
- added D26: D, Diode_SMD:D_SOD-123, B.Cu at (220.1, 124.6)
- added D27: D, Diode_SMD:D_SOD-123, B.Cu at (239.2, 124.6)
- added D28: D, Diode_SMD:D_SOD-123, B.Cu at (258.2, 124.6)
- added D29: D, Diode_SMD:D_SOD-123, B.Cu at (277.3, 124.6)
- added D3: D, Diode_SMD:D_SOD-123, B.Cu at (105.8, 96.1)
- added D30: D, Diode_SMD:D_SOD-123, B.Cu at (305.8, 124.6)
- added D31: D, Diode_SMD:D_SOD-123, B.Cu at (339.2, 124.6)
- added D32: D, Diode_SMD:D_SOD-123, B.Cu at (358.2, 124.6)
- added D33: D, Diode_SMD:D_SOD-123, B.Cu at (377.3, 124.6)
- added D34: D, Diode_SMD:D_SOD-123, B.Cu at (53.5, 143.5)
- added D35: D, Diode_SMD:D_SOD-123, B.Cu at (77.3, 143.5)
- added D36: D, Diode_SMD:D_SOD-123, B.Cu at (96.4, 143.5)
- added D37: D, Diode_SMD:D_SOD-123, B.Cu at (115.5, 143.6)
- added D38: D, Diode_SMD:D_SOD-123, B.Cu at (134.5, 143.6)
- added D39: D, Diode_SMD:D_SOD-123, B.Cu at (153.6, 143.6)
- added D4: D, Diode_SMD:D_SOD-123, B.Cu at (124.9, 96.1)
- added D40: D, Diode_SMD:D_SOD-123, B.Cu at (172.6, 143.6)
- added D41: D, Diode_SMD:D_SOD-123, B.Cu at (191.7, 143.6)
- added D42: D, Diode_SMD:D_SOD-123, B.Cu at (210.7, 143.6)
- added D43: D, Diode_SMD:D_SOD-123, B.Cu at (229.8, 143.6)
- added D44: D, Diode_SMD:D_SOD-123, B.Cu at (248.8, 143.6)
- added D45: D, Diode_SMD:D_SOD-123, B.Cu at (267.9, 143.6)
- added D46: D, Diode_SMD:D_SOD-123, B.Cu at (286.9, 143.6)
- added D47: D, Diode_SMD:D_SOD-123, B.Cu at (310.7, 143.6)
- added D48: D, Diode_SMD:D_SOD-123, B.Cu at (339.3, 143.4)
- added D49: D, Diode_SMD:D_SOD-123, B.Cu at (358.3, 143.4)
- added D5: D, Diode_SMD:D_SOD-123, B.Cu at (143.9, 96.1)
- added D50: D, Diode_SMD:D_SOD-123, B.Cu at (377.4, 143.4)
- added D51: D, Diode_SMD:D_SOD-123, B.Cu at (55.9, 162.6)
- added D52: D, Diode_SMD:D_SOD-123, B.Cu at (82.1, 162.6)
- added D53: D, Diode_SMD:D_SOD-123, B.Cu at (101.1, 162.6)
- added D54: D, Diode_SMD:D_SOD-123, B.Cu at (120.2, 162.5)
- added D55: D, Diode_SMD:D_SOD-123, B.Cu at (139.2, 162.5)
- added D56: D, Diode_SMD:D_SOD-123, B.Cu at (158.3, 162.5)
- added D57: D, Diode_SMD:D_SOD-123, B.Cu at (177.3, 162.5)
- added D58: D, Diode_SMD:D_SOD-123, B.Cu at (196.4, 162.5)
- added D59: D, Diode_SMD:D_SOD-123, B.Cu at (215.4, 162.5)
- added D6: D, Diode_SMD:D_SOD-123, B.Cu at (172.5, 96.1)
- added D60: D, Diode_SMD:D_SOD-123, B.Cu at (234.5, 162.5)
- added D61: D, Diode_SMD:D_SOD-123, B.Cu at (253.5, 162.5)
- added D62: D, Diode_SMD:D_SOD-123, B.Cu at (272.6, 162.5)
- added D63: D, Diode_SMD:D_SOD-123, B.Cu at (303.6, 162.5)
- added D64: D, Diode_SMD:D_SOD-123, B.Cu at (60.7, 181.6)
- added D65: D, Diode_SMD:D_SOD-123, B.Cu at (91.5, 182.4)
- added D66: D, Diode_SMD:D_SOD-123, B.Cu at (110.6, 182.4)
- added D67: D, Diode_SMD:D_SOD-123, B.Cu at (129.6, 182.4)
- added D68: D, Diode_SMD:D_SOD-123, B.Cu at (148.7, 183.0)
- added D69: D, Diode_SMD:D_SOD-123, B.Cu at (167.7, 183.0)
- added D7: D, Diode_SMD:D_SOD-123, B.Cu at (191.5, 96.1)
- added D70: D, Diode_SMD:D_SOD-123, B.Cu at (186.8, 183.0)
- added D71: D, Diode_SMD:D_SOD-123, B.Cu at (205.8, 183.0)
- added D72: D, Diode_SMD:D_SOD-123, B.Cu at (224.9, 183.0)
- added D73: D, Diode_SMD:D_SOD-123, B.Cu at (243.9, 183.0)
- added D74: D, Diode_SMD:D_SOD-123, B.Cu at (263.0, 183.0)
- added D75: D, Diode_SMD:D_SOD-123, B.Cu at (298.7, 183.0)
- added D76: D, Diode_SMD:D_SOD-123, B.Cu at (358.4, 182.0)
- added D77: D, Diode_SMD:D_SOD-123, B.Cu at (51.1, 200.7)
- added D78: D, Diode_SMD:D_SOD-123, B.Cu at (74.9, 201.5)
- added D79: D, Diode_SMD:D_SOD-123, B.Cu at (98.7, 201.5)
- added D8: D, Diode_SMD:D_SOD-123, B.Cu at (210.6, 96.1)
- added D80: D, Diode_SMD:D_SOD-123, B.Cu at (170.1, 202.1)
- added D81: D, Diode_SMD:D_SOD-123, B.Cu at (241.6, 202.1)
- added D82: D, Diode_SMD:D_SOD-123, B.Cu at (265.4, 202.1)
- added D83: D, Diode_SMD:D_SOD-123, B.Cu at (289.2, 202.1)
- added D84: D, Diode_SMD:D_SOD-123, B.Cu at (313.0, 202.1)
- added D85: D, Diode_SMD:D_SOD-123, B.Cu at (339.3, 201.1)
- added D86: D, Diode_SMD:D_SOD-123, B.Cu at (358.4, 201.1)
- added D87: D, Diode_SMD:D_SOD-123, B.Cu at (377.4, 201.1)
- added D9: D, Diode_SMD:D_SOD-123, B.Cu at (229.6, 96.1)
- added H1: MountingHole_Pad, MountingHole:MountingHole_3.2mm_M3_DIN965_Pad, F.Cu at (383.0, 54.4)
- added H2: MountingHole_Pad, MountingHole:MountingHole_3.2mm_M3_DIN965_Pad, F.Cu at (383.0, 71.4)
- added H3: MountingHole_Pad, MountingHole:MountingHole_3.2mm_M3_DIN965_Pad, F.Cu at (257.5, 54.7)
- added H4: MountingHole_Pad, MountingHole:MountingHole_3.2mm_M3_DIN965_Pad, F.Cu at (32.5, 216.0)
- added H5: MountingHole_Pad, MountingHole:MountingHole_3.2mm_M3_DIN965_Pad, F.Cu at (33.0, 72.4)
- added H6: MountingHole_Pad, MountingHole:MountingHole_3.2mm_M3_DIN965_Pad, F.Cu at (257.5, 70.9)
- added H7: MountingHole_Pad, MountingHole:MountingHole_3.2mm_M3_DIN965_Pad, F.Cu at (208.0, 216.0)
- added H8: MountingHole_Pad, MountingHole:MountingHole_3.2mm_M3_DIN965_Pad, F.Cu at (383.0, 216.0)
- added H9: MountingHole_Pad, MountingHole:MountingHole_3.2mm_M3_DIN965_Pad, F.Cu at (33.0, 54.4)
- added J1: 1054500101, myLibrary:MOLEX_1054500101, F.Cu at (61.8, 51.2)
- added J2: BOOT, Connector_PinHeader_2.54mm:PinHeader_1x02_P2.54mm_Horizontal, F.Cu at (151.9, 72.1)
- added J5: 10x1mm FFC/FPC, Connector_FFC-FPC:Molex_200528-0100_1x10-1MP_P1.00mm_Horizontal, F.Cu at (83.3, 59.6)
- added R1: 10k, Resistor_SMD:R_0603_1608Metric, F.Cu at (197.0, 58.9)
- added R2: 10k, Resistor_SMD:R_0603_1608Metric, F.Cu at (200.6, 58.9)
- added R3: 10k, Resistor_SMD:R_0603_1608Metric, F.Cu at (207.9, 58.9)
- added R4: 10k, Resistor_SMD:R_0603_1608Metric, F.Cu at (204.3, 58.9)
- added R5: 10K, Resistor_SMD:R_0603_1608Metric, F.Cu at (146.1, 72.6)
- added SW1: esc, myLibrary:MX_PCB_1.00u, F.Cu at (43.6, 92.2)
- added SW10: f9, myLibrary:MX_PCB_1.00u, F.Cu at (253.2, 92.2)
- added SW11: f10, myLibrary:MX_PCB_1.00u, F.Cu at (272.2, 92.2)
- added SW12: f11, myLibrary:MX_PCB_1.00u, F.Cu at (291.3, 92.2)
- added SW13: f12, myLibrary:MX_PCB_1.00u, F.Cu at (310.3, 92.2)
- added SW14: prtsc, myLibrary:MX_PCB_1.00u, F.Cu at (334.2, 92.2)
- added SW15: scroll lock, myLibrary:MX_PCB_1.00u, F.Cu at (353.2, 92.2)
- added SW16: pause break, myLibrary:MX_PCB_1.00u, F.Cu at (372.3, 92.2)
- added SW17: ~ `, myLibrary:MX_PCB_1.00u, F.Cu at (43.6, 120.8)
- added SW18: ! 1, myLibrary:MX_PCB_1.00u, F.Cu at (62.7, 120.8)
- added SW19: @ 2, myLibrary:MX_PCB_1.00u, F.Cu at (81.7, 120.8)
- added SW2: f1, myLibrary:MX_PCB_1.00u, F.Cu at (81.7, 92.2)
- added SW20: # 3, myLibrary:MX_PCB_1.00u, F.Cu at (100.8, 120.8)
- added SW21: $ 4, myLibrary:MX_PCB_1.00u, F.Cu at (119.8, 120.8)
- added SW22: % 5, myLibrary:MX_PCB_1.00u, F.Cu at (138.9, 120.8)
- added SW23: ^ 6, myLibrary:MX_PCB_1.00u, F.Cu at (157.9, 120.8)
- added SW24: & 7, myLibrary:MX_PCB_1.00u, F.Cu at (177.0, 120.8)
- added SW25: * 8, myLibrary:MX_PCB_1.00u, F.Cu at (196.0, 120.8)
- added SW26: ( 9, myLibrary:MX_PCB_1.00u, F.Cu at (215.1, 120.8)
- added SW27: ) 0, myLibrary:MX_PCB_1.00u, F.Cu at (234.1, 120.8)
- added SW28: - _, myLibrary:MX_PCB_1.00u, F.Cu at (253.2, 120.8)
- added SW29: + =, myLibrary:MX_PCB_1.00u, F.Cu at (272.2, 120.8)
- added SW3: f2, myLibrary:MX_PCB_1.00u, F.Cu at (100.8, 92.2)
- added SW30: backspace, myLibrary:MX_PCB_2.00u, F.Cu at (300.8, 120.8)
- added SW31: insert, myLibrary:MX_PCB_1.00u, F.Cu at (334.2, 120.8)
- added SW32: home, myLibrary:MX_PCB_1.00u, F.Cu at (353.2, 120.8)
- added SW33: pgup, myLibrary:MX_PCB_1.00u, F.Cu at (372.3, 120.8)
- added SW34: tab, myLibrary:MX_PCB_1.50u, F.Cu at (48.4, 139.8)
- added SW35: q, myLibrary:MX_PCB_1.00u, F.Cu at (72.2, 139.8)
- added SW36: w, myLibrary:MX_PCB_1.00u, F.Cu at (91.3, 139.8)
- added SW37: e, myLibrary:MX_PCB_1.00u, F.Cu at (110.3, 139.8)
- added SW38: r, myLibrary:MX_PCB_1.00u, F.Cu at (129.4, 139.8)
- added SW39: t, myLibrary:MX_PCB_1.00u, F.Cu at (148.4, 139.8)
- added SW4: f3, myLibrary:MX_PCB_1.00u, F.Cu at (119.8, 92.2)
- added SW40: y, myLibrary:MX_PCB_1.00u, F.Cu at (167.5, 139.8)
- added SW41: u, myLibrary:MX_PCB_1.00u, F.Cu at (186.5, 139.8)
- added SW42: I, myLibrary:MX_PCB_1.00u, F.Cu at (205.6, 139.8)
- added SW43: O, myLibrary:MX_PCB_1.00u, F.Cu at (224.6, 139.8)
- added SW44: P, myLibrary:MX_PCB_1.00u, F.Cu at (243.7, 139.8)
- added SW45: { [, myLibrary:MX_PCB_1.00u, F.Cu at (262.7, 139.8)
- added SW46: } ], myLibrary:MX_PCB_1.00u, F.Cu at (281.8, 139.8)
- added SW47: | \, myLibrary:MX_PCB_1.50u, F.Cu at (305.6, 139.8)
- added SW48: delete, myLibrary:MX_PCB_1.00u, F.Cu at (334.2, 139.8)
- added SW49: end, myLibrary:MX_PCB_1.00u, F.Cu at (353.2, 139.8)
- added SW5: f4, myLibrary:MX_PCB_1.00u, F.Cu at (138.9, 92.2)
- added SW50: pgdn, myLibrary:MX_PCB_1.00u, F.Cu at (372.3, 139.8)
- added SW51: caps lock, myLibrary:MX_PCB_1.00u, F.Cu at (50.8, 158.9)
- added SW52: a, myLibrary:MX_PCB_1.00u, F.Cu at (77.0, 158.9)
- added SW53: s, myLibrary:MX_PCB_1.00u, F.Cu at (96.0, 158.9)
- added SW54: d, myLibrary:MX_PCB_1.00u, F.Cu at (115.1, 158.9)
- added SW55: f, myLibrary:MX_PCB_1.00u, F.Cu at (134.1, 158.9)
- added SW56: g, myLibrary:MX_PCB_1.00u, F.Cu at (153.2, 158.9)
- added SW57: h, myLibrary:MX_PCB_1.00u, F.Cu at (172.2, 158.9)
- added SW58: j, myLibrary:MX_PCB_1.00u, F.Cu at (191.3, 158.9)
- added SW59: K, myLibrary:MX_PCB_1.00u, F.Cu at (210.3, 158.9)
- added SW6: f5, myLibrary:MX_PCB_1.00u, F.Cu at (167.5, 92.2)
- added SW60: L, myLibrary:MX_PCB_1.00u, F.Cu at (229.4, 158.9)
- added SW61: : ;, myLibrary:MX_PCB_1.00u, F.Cu at (248.4, 158.9)
- added SW62: " ', myLibrary:MX_PCB_1.00u, F.Cu at (267.5, 158.9)
- added SW63: enter, myLibrary:MX_PCB_2.25u, F.Cu at (298.4, 158.9)
- added SW64: lshift, myLibrary:MX_PCB_2.25u, F.Cu at (55.6, 177.9)
- added SW65: z, myLibrary:MX_PCB_1.00u, F.Cu at (86.5, 177.9)
- added SW66: x, myLibrary:MX_PCB_1.00u, F.Cu at (105.6, 177.9)
- added SW67: c, myLibrary:MX_PCB_1.00u, F.Cu at (124.6, 177.9)
- added SW68: v, myLibrary:MX_PCB_1.00u, F.Cu at (143.7, 177.9)
- added SW69: b, myLibrary:MX_PCB_1.00u, F.Cu at (162.7, 177.9)
- added SW7: f6, myLibrary:MX_PCB_1.00u, F.Cu at (186.5, 92.2)
- added SW70: n, myLibrary:MX_PCB_1.00u, F.Cu at (181.8, 177.9)
- added SW71: m, myLibrary:MX_PCB_1.00u, F.Cu at (200.8, 177.9)
- added SW72: < ,, myLibrary:MX_PCB_1.00u, F.Cu at (219.9, 177.9)
- added SW73: > ., myLibrary:MX_PCB_1.00u, F.Cu at (238.9, 177.9)
- added SW74: ? /, myLibrary:MX_PCB_1.00u, F.Cu at (258.0, 177.9)
- added SW75: rshift, myLibrary:MX_PCB_2.75u, F.Cu at (293.7, 177.9)
- added SW76: uparrow, myLibrary:MX_PCB_1.00u, F.Cu at (353.2, 177.9)
- added SW77: lctrl, myLibrary:MX_PCB_1.25u, F.Cu at (46.0, 197.0)
- added SW78: lwin, myLibrary:MX_PCB_1.25u, F.Cu at (69.8, 197.0)
- added SW79: lalt, myLibrary:MX_PCB_1.25u, F.Cu at (93.7, 197.0)
- added SW8: f7, myLibrary:MX_PCB_1.00u, F.Cu at (205.6, 92.2)
- added SW80: spacebar, myLibrary:MX_PCB_6.25u, F.Cu at (165.1, 197.0)
- added SW81: ralt, myLibrary:MX_PCB_1.25u, F.Cu at (236.5, 197.0)
- added SW82: Win, myLibrary:MX_PCB_1.25u, F.Cu at (260.3, 197.0)
- added SW83: Menu, myLibrary:MX_PCB_1.25u, F.Cu at (284.2, 197.0)
- added SW84: rctrl, myLibrary:MX_PCB_1.25u, F.Cu at (308.0, 197.0)
- added SW85: leftarrow, myLibrary:MX_PCB_1.00u, F.Cu at (334.2, 197.0)
- added SW86: downarrow, myLibrary:MX_PCB_1.00u, F.Cu at (353.2, 197.0)
- added SW87: rightarrow, myLibrary:MX_PCB_1.00u, F.Cu at (372.3, 197.0)
- added SW9: f8, myLibrary:MX_PCB_1.00u, F.Cu at (224.6, 92.2)
- added U1: ESP32-S3-WROOM-1-N16R8, myLibrary:ESP32-S3-WROOM-1_EXP, F.Cu at (118.3, 64.1)
- added U2: MCP1825S-2502E/DB, myLibrary:SOT-223_3MC_MCH, F.Cu at (153.3, 61.1)
Other:
- board outline added: 358.6 x 171.8 mm

Commit message: started pcb routing, 63 connections left
Parts:
- U1: moved to B.Cu
- moved U1 171.7 mm to (290.1, 63.2), turned to 180 degrees
- moved J2 39.1 mm to (115.0, 59.1)
- moved R5 14.7 mm to (138.4, 60.1), turned to 0 degrees
Routing:
- net GND: track 0.00 -> 847.5 mm
- net /keyboard_matrix/row_5: track 0.00 -> 590.7 mm
- net /keyboard_matrix/row_4: track 0.00 -> 535.2 mm
- net /keyboard_matrix/row_0: track 0.00 -> 510.3 mm
- net /keyboard_matrix/row_3: track 0.00 -> 506.6 mm
- net /keyboard_matrix/row_2: track 0.00 -> 498.3 mm
- net /keyboard_matrix/row_1: track 0.00 -> 484.6 mm
- net /keyboard_matrix/col_4: track 0.00 -> 258.6 mm
- net /keyboard_matrix/col_5: track 0.00 -> 257.8 mm
- net /keyboard_matrix/col_6: track 0.00 -> 220.3 mm
- net /keyboard_matrix/col_8: track 0.00 -> 215.1 mm
- net /keyboard_matrix/col_7: track 0.00 -> 203.4 mm
- net /keyboard_matrix/col_9: track 0.00 -> 198.8 mm
- net /keyboard_matrix/col_16: track 0.00 -> 193.3 mm
- net /keyboard_matrix/col_13: track 0.00 -> 173.8 mm, vias 0 -> 1
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Other:
- board size 358.6 x 171.8 mm -> 361.4 x 171.8 mm

Commit message: keyboard routing done, lipo remaining
Parts:
- moved R3 29.0 mm to (178.9, 59.2), turned to 90 degrees
- moved CR1 16.9 mm to (77.4, 55.5), turned to 0 degrees
- moved C1 14.6 mm to (191.3, 59.2)
- moved R2 12.4 mm to (188.2, 59.2)
- moved R1 11.9 mm to (185.1, 59.2)
- moved J5 10.6 mm to (93.0, 55.4)
- moved R4 9.82 mm to (194.4, 59.2)
- moved C4 8.08 mm to (175.8, 59.2)
- moved R5 6.87 mm to (131.6, 60.1), turned to 90 degrees
- moved J1 1.98 mm to (61.9, 49.2)
- moved C5 1.74 mm to (182.0, 59.2)
- moved C2 0.54 mm to (172.7, 59.2)
- moved C3 0.28 mm to (169.6, 59.2)
Routing:
- net +3V3: track 0.00 -> 385.6 mm, vias 0 -> 4
- net /D-: track 0.00 -> 322.6 mm, vias 0 -> 3
- net /D+: track 0.00 -> 292.9 mm, vias 0 -> 1
- net /CC2: track 0.00 -> 262.5 mm, vias 0 -> 6
- net GND: track 847.5 -> 1102.3 mm, vias 0 -> 8
- net /CC1: track 0.00 -> 251.4 mm, vias 0 -> 4
- net /keyboard_matrix/col_0: track 113.7 -> 363.0 mm, vias 0 -> 1
- net /keyboard_matrix/col_1: track 129.8 -> 340.5 mm, vias 0 -> 1
- net Net-(J1-SHIELD1): track 0.00 -> 207.9 mm, vias 0 -> 5
- net /TX: track 0.00 -> 200.3 mm, vias 0 -> 1
- net /RX: track 0.00 -> 198.8 mm, vias 0 -> 3
- net Net-(J2-Pin_2): track 0.00 -> 192.6 mm, vias 0 -> 1
- net /keyboard_matrix/col_2: track 127.5 -> 318.6 mm, vias 0 -> 1
- net /keyboard_matrix/col_3: track 103.5 -> 289.2 mm, vias 0 -> 3
- net Net-(U1-EN): track 0.00 -> 180.5 mm, vias 0 -> 3
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